File: _autosave-riscy.kicad_sch (KiCad schematic)
At the start: 38 parts, among them J1 Conn_01x15_Pin, J2 Conn_01x15_Pin, J3 USB_C_Receptacle_USB2.0_14P, Q1 MMBT2222A, Q2 MMBT2222A, SW1 SW_Push, SW2 SW_Push, U2 FT231XS, U3 ESP32-C3-WROOM-02, U4 AMS1117-3.3

Commit message: updated schematic
Connections:
- net +3V3: no longer C4.1, U2.13 (3V3OUT), U2.14 (~{RESET}), U2.3 (VCCIO)
- net +5V: now also R2.1, U4.3 (VI)
- net IO9: now also Q2.2 (E)
- new net 3v3: C4.1, U2.13 (3V3OUT), U2.14 (~{RESET}), U2.3 (VCCIO)
- no-connect marks 4 -> 6
Changed lines of the file:
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@@
 	)
 	(junction
+		(at 328.93 163.83)
+		(diameter 0)
+		(color 0 0 0 0)
+	)
+	(junction
 		(at 347.98 182.88)
 		(diameter 0)
@@
 	)
 	(junction
+		(at 77.47 45.72)
+		(diameter 0)
+		(color 0 0 0 0)
+	)
+	(junction
 		(at 293.37 48.26)
 		(diameter 0)
@@
 	)
 	(no_connect
+		(at 185.42 76.2)
+	)
+	(no_connect
 		(at 185.42 53.34)
 	)
 	(no_connect
+		(at 185.42 68.58)
+	)
+	(no_connect
 		(at 185.42 63.5)
 	)
@@
 	(wire
 		(pts
-			(xy 313.69 163.83) (xy 340.36 163.83)
+			(xy 313.69 163.83) (xy 328.93 163.83)
 		)
 		(stroke
@@
 	(wire
 		(pts
+			(xy 328.93 163.83) (xy 328.93 167.64)
+		)
+		(stroke
+			(width 0)
+			(type default)
+		)
+	)
+	(wire
+		(pts
 			(xy 191.77 144.78) (xy 199.39 144.78)
 		)
@@
 	(wire
 		(pts
+			(xy 328.93 158.75) (xy 328.93 163.83)
+		)
+		(stroke
+			(width 0)
+			(type default)
+		)
+	)
+	(wire
+		(pts
 			(xy 153.67 146.05) (xy 158.75 146.05)
 		)
@@
 	(wire
 		(pts
-			(xy 328.93 158.75) (xy 328.93 167.64)
-		)
-		(stroke
-			(width 0)
-			(type default)
-		)
-	)
-	(wire
-		(pts
 			(xy 261.62 151.13) (xy 270.51 151.13)
 		)
@@
 	(wire
 		(pts
+			(xy 328.93 163.83) (xy 340.36 163.83)
+		)
+		(stroke
+			(width 0)
+			(type default)
+		)
+	)
+	(wire
+		(pts
 			(xy 355.6 163.83) (xy 377.19 163.83)
 		)
@@
 	)
 	(label "VCCIO"
-		(at 27.94 50.8 180)
+		(at 27.94 45.72 180)
 		(effects
 			(font
@@
 		)
 	)
+	(label "IO9"
+		(at 99.06 146.05 0)
+		(effects
+			(font
+				(size 1.27 1.27)
+			)
+			(justify left bottom)
+		)
+	)
 	(label "U0RXD"
 		(at 207.01 52.07 0)
@@
 	)
 	(symbol
-		(lib_id "power:+3V3")
-		(at 27.94 45.72 0)
-		(unit 1)
-		(exclude_from_sim no)
-		(in_bom yes)
-		(on_board yes)
-		(dnp no)
-		(fields_autoplaced yes)
-		(property "Reference" "#PWR017"
-			(at 27.94 49.53 0)
-			(effects
-				(font
-					(size 1.27 1.27)
-				)
-				(hide yes)
-			)
-		)
-		(property "Value" "+3V3"
-			(at 27.94 40.64 0)
-			(effects
-				(font
-					(size 1.27 1.27)
-				)
-			)
-		)
-		(property "Footprint" ""
-			(at 27.94 45.72 0)
-			(effects
-				(font
-					(size 1.27 1.27)
-				)
-				(hide yes)
-			)
-		)
-		(property "Datasheet" ""
-			(at 27.94 45.72 0)
-			(effects
-				(font
-					(size 1.27 1.27)
-				)
-				(hide yes)
-			)
-		)
-		(property "Description" "Power symbol creates a global label with name \"+3V3\""
-			(at 27.94 45.72 0)
-			(effects
-				(font
-					(size 1.27 1.27)
-				)
-				(hide yes)
-			)
-		)
-		(pin "1"
-		)
-		(instances
-			(project ""
-				(path "/de2d24e1-940f-49f9-a4cc-0c6b868ad501"
-					(reference "#PWR017")
-					(unit 1)
-				)
-			)
-		)
-	)
-	(symbol
 		(lib_id "Device:R")
 		(at 198.12 43.18 90)
@@
 					(unit 1)
 				)
+			)
+		)
+	)
+	(symbol
+		(lib_id "power:PWR_FLAG")
+		(at 77.47 45.72 0)
+		(unit 1)
+		(exclude_from_sim no)
+		(in_bom yes)
+		(on_board yes)
+		(dnp no)
+		(fields_autoplaced yes)
+		(property "Reference" "#FLG01"
+			(at 77.47 43.815 0)
+			(effects
+				(font
+					(size 1.27 1.27)
+				)
+				(hide yes)
+			)
+		)
+		(property "Value" "PWR_FLAG"
+			(at 77.47 40.64 0)
+			(effects
+				(font
+					(size 1.27 1.27)
+				)
+			)
+		)
+		(property "Footprint" ""
+			(at 77.47 45.72 0)
+			(effects
+				(font
+					(size 1.27 1.27)
+				)
+				(hide yes)
+			)
+		)
+		(property "Datasheet" "~"
+			(at 77.47 45.72 0)
+			(effects
+				(font
+					(size 1.27 1.27)
+				)
+				(hide yes)
+			)
+		)
+		(property "Description" "Special symbol for telling ERC where power comes from"
+			(at 77.47 45.72 0)
+			(effects
+				(font
+					(size 1.27 1.27)
+				)
+				(hide yes)
+			)
+		)
+		(pin "1"
+		)
+		(instances
+			(project ""
+				(path "/de2d24e1-940f-49f9-a4cc-0c6b868ad501"
+					(reference "#FLG01")
+					(unit 1)
+				)
