File: riscy.kicad_sch (KiCad schematic)
At the start: 38 parts, among them J1 Conn_01x15_Pin, J2 Conn_01x15_Pin, J3 USB_C_Receptacle_USB2.0_14P, Q1 MMBT2222A, Q2 MMBT2222A, SW1 SW_MEC_5E, SW3 SW_MEC_5E, U2 FT231XS, U3 ESP32-C3-WROOM-02, U4 AMS1117-3.3

Commit message: changed schematics
Parts:
- C3: footprint Capacitor_SMD:C_0805_2012Metric -> Capacitor_SMD:C_1206_3216Metric
Changed lines of the file:
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@@
 			)
 		)
-		(property "Footprint" "Capacitor_SMD:C_0805_2012Metric"
+		(property "Footprint" "Capacitor_SMD:C_1206_3216Metric"
 			(at 272.7452 60.96 0)
 			(effects

Commit message: changed schematics
Changed lines of the file:
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@@
 	)
 	(junction
+		(at 345.44 85.09)
+		(diameter 0)
+		(color 0 0 0 0)
+	)
+	(junction
 		(at 77.47 59.69)
 		(diameter 0)
@@
 					(unit 1)
 				)
+			)
+		)
+	)
+	(symbol
+		(lib_id "power:PWR_FLAG")
+		(at 345.44 85.09 90)
+		(unit 1)
+		(exclude_from_sim no)
+		(in_bom yes)
+		(on_board yes)
+		(dnp no)
+		(fields_autoplaced yes)
+		(property "Reference" "#FLG02"
+			(at 343.535 85.09 0)
+			(effects
+				(font
+					(size 1.27 1.27)
+				)
+				(hide yes)
+			)
+		)
+		(property "Value" "PWR_FLAG"
+			(at 341.63 85.0899 90)
+			(effects
+				(font
+					(size 1.27 1.27)
+				)
+				(justify left)
+			)
+		)
+		(property "Footprint" ""
+			(at 345.44 85.09 0)
+			(effects
+				(font
+					(size 1.27 1.27)
+				)
+				(hide yes)
+			)
+		)
+		(property "Datasheet" "~"
+			(at 345.44 85.09 0)
+			(effects
+				(font
+					(size 1.27 1.27)
+				)
+				(hide yes)
+			)
+		)
+		(property "Description" "Special symbol for telling ERC where power comes from"
+			(at 345.44 85.09 0)
+			(effects
+				(font
+					(size 1.27 1.27)
+				)
+				(hide yes)
+			)
+		)
+		(pin "1"
+		)
+		(instances
+			(project ""
+				(path "/de2d24e1-940f-49f9-a4cc-0c6b868ad501"
+					(reference "#FLG02")
+					(unit 1)
+				)

Commit message: making pcb
Parts:
- removed D2, D3: LED, LED_SMD:LED_2010_5025Metric, symbol Device:LED
Connections:
- net +3V3: now also R4.2, R5.2
Changed lines of the file:
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@@
 	(wire
 		(pts
-			(xy 205.74 71.12) (xy 215.9 71.12)
+			(xy 205.74 71.12) (xy 223.52 71.12)
 		)
 		(stroke
@@
 	(wire
 		(pts
-			(xy 213.36 73.66) (xy 213.36 78.74)
+			(xy 213.36 73.66) (xy 213.36 86.36)
 		)
 		(stroke
@@
 	)
 	(symbol
-		(lib_id "Device:LED")
-		(at 213.36 82.55 270)
-		(unit 1)
-		(exclude_from_sim no)
-		(in_bom yes)
-		(on_board yes)
-		(dnp no)
-		(fields_autoplaced yes)
-		(property "Reference" "D3"
-			(at 215.9 79.6924 90)
-			(effects
-				(font
-					(size 1.27 1.27)
-				)
-				(justify left)
-			)
-		)
-		(property "Value" "LED"
-			(at 215.9 82.2324 90)
-			(effects
-				(font
-					(size 1.27 1.27)
-				)
-				(justify left)
-			)
-		)
-		(property "Footprint" "LED_SMD:LED_2010_5025Metric"
-			(at 213.36 82.55 0)
-			(effects
-				(font
-					(size 1.27 1.27)
-				)
-				(hide yes)
-			)
-		)
-		(property "Datasheet" "~"
-			(at 213.36 82.55 0)
-			(effects
-				(font
-					(size 1.27 1.27)
-				)
-				(hide yes)
-			)
-		)
-		(property "Description" "Light emitting diode"
-			(at 213.36 82.55 0)
-			(effects
-				(font
-					(size 1.27 1.27)
-				)
-				(hide yes)
-			)
-		)
-		(pin "1"
-		)
-		(pin "2"
-		)
-		(instances
-			(project "riscy"
-				(path "/de2d24e1-940f-49f9-a4cc-0c6b868ad501"
-					(reference "D3")
-					(unit 1)
-				)
-			)
-		)
-	)
-	(symbol
 		(lib_id "Jumper:SolderJumper_2_Open")
 		(at 200.66 73.66 180)
@@
 					(unit 1)
 				)
-			)
-		)
-	)
-	(symbol
-		(lib_id "Device:LED")
-		(at 219.71 71.12 0)
-		(unit 1)
-		(exclude_from_sim no)
-		(in_bom yes)
-		(on_board yes)
-		(dnp no)
-		(fields_autoplaced yes)
-		(property "Reference" "D2"
-			(at 218.1225 64.77 0)
-			(effects
-				(font
-					(size 1.27 1.27)
-				)
-			)
-		)
-		(property "Value" "LED"
-			(at 218.1225 67.31 0)
-			(effects
-				(font
-					(size 1.27 1.27)
-				)
-			)
-		)
-		(property "Footprint" "LED_SMD:LED_2010_5025Metric"
-			(at 219.71 71.12 0)
-			(effects
-				(font
-					(size 1.27 1.27)
-				)
-				(hide yes)
-			)
-		)
-		(property "Datasheet" "~"
-			(at 219.71 71.12 0)
-			(effects
-				(font
-					(size 1.27 1.27)
-				)
-				(hide yes)
-			)
-		)
-		(property "Description" "Light emitting diode"
-			(at 219.71 71.12 0)
-			(effects
-				(font
-					(size 1.27 1.27)
-				)
-				(hide yes)
-			)
-		)
-		(pin "1"
-		)
-		(pin "2"
-		)
-		(instances
-			(project ""
-				(path "/de2d24e1-940f-49f9-a4cc-0c6b868ad501"
-					(reference "D2")
-					(unit 1)
-				)

Commit message: updated
Changed lines of the file:
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@@
 (kicad_sch
-	(version 20231120)
+	(version 20250114)
 	(generator "eeschema")
-	(generator_version "8.0")
+	(generator_version "9.0")
 	(paper "A3")
 	(title_block
@@
 		(date "7/01/25")
 	)
+	(rectangle
+		(start 29.845 149.225)
+		(end 52.705 163.195)
+		(stroke
+			(width 0)
+			(type solid)
+			(color 255 160 107 1)
+		)
+		(fill
+			(type none)
+		)
+	)
+	(rectangle
+		(start 249.555 21.59)
+		(end 391.795 100.965)
+		(stroke
+			(width 0)
+			(type dash_dot)
+			(color 130 161 255 1)
+		)
+		(fill
+			(type none)
+		)
+	)
+	(rectangle
+		(start 18.415 107.95)
+		(end 114.935 171.45)
+		(stroke
+			(width 0)
+			(type dash_dot)
+			(color 130 161 255 1)
+		)
+		(fill
+			(type none)
+		)
+	)
+	(rectangle
+		(start 299.085 140.335)
+		(end 395.605 203.835)
+		(stroke
+			(width 0)
+			(type dash_dot)
+			(color 130 161 255 1)
+		)
+		(fill
+			(type none)
+		)
+	)
+	(rectangle
+		(start 18.415 22.86)
+		(end 237.49 102.235)
+		(stroke
+			(width 0)
+			(type dash_dot)
+			(color 130 161 255 1)
+		)
+		(fill
+			(type none)
+		)
+	)
+	(rectangle
+		(start 298.45 107.95)
+		(end 375.285 133.35)
+		(stroke
+			(width 0)
+			(type dash_dot)
+			(color 130 161 255 1)
+		)
+		(fill
+			(type none)
+		)
+	)
+	(rectangle
+		(start 123.825 107.95)
+		(end 220.345 171.45)
+		(stroke
+			(width 0)
+			(type dash_dot)
+			(color 130 161 255 1)
+		)
+		(fill
+			(type none)
+		)
+	)
+	(rectangle
+		(start 231.14 107.95)
+		(end 288.925 171.45)
+		(stroke
+			(width 0)
+			(type dash_dot)
+			(color 130 161 255 1)
+		)
+		(fill
+			(type none)
+		)
+	)
+	(text "USB-C to UART"
+		(exclude_from_sim no)
+		(at 35.814 28.448 0)
+		(effects
+			(font
+				(face "JetBrains Mono SemiBold")
+				(size 2.54 2.54)
+				(color 101 200 99 1)
+			)
+		)
+	)
+	(text "DTR RTS-->EN IO0\n1 	1 	   1  1\n0    0 	   1  1\n1 	0	   0  1\n0 	1 	   1  0"
+		(exclude_from_sim no)
+		(at 41.656 156.464 0)
+		(effects
+			(font
+				(size 1.27 1.27)
+			)
+		)
+	)
+	(text "Voltage Regulator"
+		(exclude_from_sim no)
+		(at 319.278 145.542 0)
+		(effects
+			(font
+				(face "JetBrainsMono NF Medium")
+				(size 2.54 2.54)
+				(color 101 200 99 1)
+			)
+		)
+	)
+	(text "Reset and Boot buttons"
+		(exclude_from_sim no)
+		(at 255.778 112.268 0)
+		(effects
+			(font
+				(face "JetBrains Mono SemiBold")
+				(size 2.54 2.54)
+				(color 101 200 99 1)
+			)
+		)
+	)
+	(text "Sphuro"
+		(exclude_from_sim no)
+		(at 332.486 263.906 0)
+		(effects
+			(font
+				(face "ArcadeClassic")
+				(size 12.7 12.7)
+				(color 59 142 217 1)
+			)
+		)
+	)
+	(text "Connector Pins"
+		(exclude_from_sim no)
+		(at 140.716 112.522 0)
+		(effects
+			(font
+				(face "JetBrains Mono SemiBold")
+				(size 2.54 2.54)
+				(color 101 200 99 1)
+			)
+		)
+	)
+	(text "ESP32-C3-wroom-02"
+		(exclude_from_sim no)
+		(at 270.256 27.178 0)
+		(effects
+			(font
+				(face "JetBrains Mono SemiBold")
+				(size 2.54 2.54)
+				(color 101 200 99 1)
+			)
+		)
+	)
+	(text "Programmable LED"
+		(exclude_from_sim no)
+		(at 317.373 112.268 0)
+		(effects
+			(font
+				(face "JetBrains Mono SemiBold")
+				(size 2.54 2.54)
+				(color 101 200 99 1)
+			)
+		)
+	)
+	(text "USB to UART programmer"
+		(exclude_from_sim no)
+		(at 43.688 113.03 0)
+		(effects
+			(font
+				(face "JetBrains Mono SemiBold")
+				(size 2.54 2.54)
+				(color 101 200 99 1)
+			)
+		)
+	)
 	(junction
 		(at 266.7 124.46)
@@
 		)
 	)
-	(rectangle
-		(start 29.845 149.225)
-		(end 52.705 163.195)
-		(stroke
-			(width 0)
-			(type solid)
-			(color 255 160 107 1)
-		)
-		(fill
-			(type none)
-		)
-	)
-	(rectangle
-		(start 249.555 21.59)
-		(end 391.795 100.965)
-		(stroke
-			(width 0)
-			(type dash_dot)
-			(color 130 161 255 1)
-		)
-		(fill
-			(type none)
-		)
-	)
-	(rectangle
-		(start 18.415 107.95)
-		(end 114.935 171.45)
-		(stroke
-			(width 0)
-			(type dash_dot)
-			(color 130 161 255 1)
-		)
-		(fill
-			(type none)
-		)
-	)
-	(rectangle
-		(start 299.085 140.335)
-		(end 395.605 203.835)
-		(stroke
-			(width 0)
-			(type dash_dot)
-			(color 130 161 255 1)
-		)
-		(fill
-			(type none)
-		)
-	)
-	(rectangle
-		(start 18.415 22.86)
-		(end 237.49 102.235)
-		(stroke
-			(width 0)
-			(type dash_dot)
-			(color 130 161 255 1)
-		)
-		(fill
-			(type none)
-		)
-	)
-	(rectangle
-		(start 298.45 107.95)
-		(end 375.285 133.35)
-		(stroke
-			(width 0)
-			(type dash_dot)
-			(color 130 161 255 1)
-		)
-		(fill
-			(type none)
-		)
-	)
-	(rectangle
-		(start 123.825 107.95)
-		(end 220.345 171.45)
-		(stroke
-			(width 0)
-			(type dash_dot)
-			(color 130 161 255 1)
-		)
-		(fill
-			(type none)
-		)
-	)
-	(rectangle
-		(start 231.14 107.95)
-		(end 288.925 171.45)
-		(stroke
-			(width 0)
-			(type dash_dot)
-			(color 130 161 255 1)
-		)
-		(fill
-			(type none)
-		)
-	)
-	(text "USB-C to UART"
-		(exclude_from_sim no)
-		(at 35.814 28.448 0)
-		(effects
-			(font
-				(face "JetBrains Mono SemiBold")
-				(size 2.54 2.54)
-				(color 101 200 99 1)
-			)
-		)
-	)
-	(text "DTR RTS-->EN IO0\n1 	1 	   1  1\n0    0 	   1  1\n1 	0	   0  1\n0 	1 	   1  0"
-		(exclude_from_sim no)
-		(at 41.656 156.464 0)
-		(effects
-			(font
-				(size 1.27 1.27)
-			)
-		)
-	)
-	(text "Voltage Regulator"
-		(exclude_from_sim no)
-		(at 319.278 145.542 0)
-		(effects
-			(font
-				(face "JetBrainsMono NF Medium")
-				(size 2.54 2.54)
-				(color 101 200 99 1)
-			)
-		)
-	)
-	(text "Reset and Boot buttons"
-		(exclude_from_sim no)
-		(at 255.778 112.268 0)
-		(effects
-			(font
-				(face "JetBrains Mono SemiBold")
-				(size 2.54 2.54)
-				(color 101 200 99 1)
-			)
-		)
-	)
-	(text "Sphuro"
-		(exclude_from_sim no)
-		(at 332.486 263.906 0)
-		(effects
-			(font
-				(face "ArcadeClassic")
-				(size 12.7 12.7)
-				(color 59 142 217 1)
-			)
-		)
-	)
-	(text "Connector Pins"
-		(exclude_from_sim no)
-		(at 140.716 112.522 0)
-		(effects
-			(font
-				(face "JetBrains Mono SemiBold")
-				(size 2.54 2.54)
-				(color 101 200 99 1)
-			)
-		)
-	)
-	(text "ESP32-C3-wroom-02"
-		(exclude_from_sim no)
-		(at 270.256 27.178 0)
-		(effects
-			(font
-				(face "JetBrains Mono SemiBold")
-				(size 2.54 2.54)
-				(color 101 200 99 1)
-			)
-		)
-	)
-	(text "Programmable LED"
-		(exclude_from_sim no)
-		(at 317.373 112.268 0)
-		(effects
-			(font
-				(face "JetBrains Mono SemiBold")
-				(size 2.54 2.54)
-				(color 101 200 99 1)
-			)
-		)
-	)
-	(text "USB to UART programmer"
-		(exclude_from_sim no)
-		(at 43.688 113.03 0)
-		(effects
-			(font
-				(face "JetBrains Mono SemiBold")
-				(size 2.54 2.54)
-				(color 101 200 99 1)
-			)
-		)
-	)
 	(label "IO6"
 		(at 330.2 64.77 180)
@@
 		)
 	)
+	(embedded_fonts no)
 )
