File: riscy.kicad_pcb (KiCad board)
At the start: 2 copper layers, 38 parts, among them J1 Conn_01x15_Pin, J2 Conn_01x15_Pin, J3 USB_C_Receptacle_USB2.0_14P, Q1 MMBT2222A, Q2 MMBT2222A, SW1 SW_MEC_5E, SW3 SW_MEC_5E, U2 FT231XS, U3 ESP32-C3-WROOM-02, U4 AMS1117-3.3

Commit message: changed
Parts:
- moved D4 142.9 mm to (54.4, 140.0)
- moved R12 111.2 mm to (48.5, 140.0)
- moved U4 22.7 mm to (52.6, 147.2)
- moved J1 21.2 mm to (43.0, 114.6)
- moved R1 17.0 mm to (59.5, 131.0)
- moved Q2 16.3 mm to (85.6, 142.5)
- moved D3 12.8 mm to (148.0, 129.5)
- moved U3 11.4 mm to (67.0, 112.2)
- moved J2 7.52 mm to (92.0, 115.0)
- moved Q1 5.52 mm to (69.5, 134.5)
Changed lines of the file:
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@@
 	(footprint "LED_SMD:LED_1206_3216Metric"
 		(layer "F.Cu")
-		(at 172.6825 59.73)
+		(at 54.4 140)
 		(descr "LED SMD 1206 (3216 Metric), square (rectangular) end terminal, IPC_7351 nominal, (Body size source: http://www.tortai-tech.com/upload/download/2011102023233369053.pdf), generated with kicad-footprint-generator")
 		(tags "LED")
@@
 	(footprint "Package_TO_SOT_SMD:SOT-223-3_TabPin2"
 		(layer "F.Cu")
-		(at 70 132.5)
+		(at 52.65 147.2)
 		(descr "module CMS SOT223 4 pins")
 		(tags "CMS SOT")
@@
 	(footprint "Resistor_SMD:R_1206_3216Metric"
 		(layer "F.Cu")
-		(at 76 127)
+		(at 59.4625 131)
 		(descr "Resistor SMD 1206 (3216 Metric), square (rectangular) end terminal, IPC_7351 nominal, (Body size source: IPC-SM-782 page 72, https://www.pcb-3d.com/wordpress/wp-content/uploads/ipc-sm-782a_amendment_1_and_2.pdf), generated with kicad-footprint-generator")
 		(tags "resistor")
@@
 	(footprint "Connector_PinHeader_2.54mm:PinHeader_1x15_P2.54mm_Vertical"
 		(layer "F.Cu")
-		(at 92 122.52)
+		(at 92 115)
 		(descr "Through hole straight pin header, 1x15, 2.54mm pitch, single row")
 		(tags "Through hole pin header THT 1x15 2.54mm single row")
@@
 	(footprint "Connector_PinHeader_2.54mm:PinHeader_1x15_P2.54mm_Vertical"
 		(layer "F.Cu")
-		(at 63 121.48)
+		(at 43 114.56)
 		(descr "Through hole straight pin header, 1x15, 2.54mm pitch, single row")
 		(tags "Through hole pin header THT 1x15 2.54mm single row")
@@
 	(footprint "Package_TO_SOT_SMD:SOT-23"
 		(layer "F.Cu")
-		(at 69.0625 140)
+		(at 69.525 134.5)
 		(descr "SOT, 3 Pin (JEDEC TO-236 Var AB https://www.jedec.org/document_search?search_api_views_fulltext=TO-236), generated with kicad-footprint-generator ipc_gullwing_generator.py")
 		(tags "SOT TO_SOT_SMD")
@@
 		(tags "SSOP 0.635")
 		(property "Reference" "U2"
-			(at 0 -5.4 360)
+			(at 0 -5.4 0)
 			(layer "F.SilkS")
 			(effects
@@
 		)
 		(property "Value" "FT231XS"
-			(at 0 5.4 360)
+			(at 0 5.4 0)
 			(layer "F.Fab")
 			(effects
@@
 		)
 		(fp_text user "${REFERENCE}"
-			(at 0 0 360)
+			(at 0 0 0)
 			(layer "F.Fab")
 			(effects
@@
 	(footprint "RF_Module:ESP32-C3-WROOM-02"
 		(layer "F.Cu")
-		(at 78.25 114)
+		(at 67.04 112.2)
 		(descr "RF Module, ESP32-C3 WROOM-02, Wi-Fi and Bluetooth, BLE, onboard antenna, https://www.espressif.com/sites/default/files/documentation/esp32-c3-wroom-02_datasheet_en.pdf")
 		(tags "ESP32-C3 WROOM-02 espressif")
@@
 			(polygon
 				(pts
-					(xy 64.25 106.9) (xy 92.25 106.9) (xy 92.25 95.9) (xy 64.25 95.9)
+					(xy 53.04 105.1) (xy 81.04 105.1) (xy 81.04 94.1) (xy 53.04 94.1)
 				)
 			)
@@
 	(footprint "LED_SMD:LED_2010_5025Metric"
 		(layer "F.Cu")
-		(at 160 125)
+		(at 148 129.5)
 		(descr "LED SMD 2010 (5025 Metric), square (rectangular) end terminal, IPC_7351 nominal, (Body size source: http://www.tortai-tech.com/upload/download/2011102023233369053.pdf), generated with kicad-footprint-generator")
 		(tags "LED")
@@
 	(footprint "Package_TO_SOT_SMD:SOT-23"
 		(layer "F.Cu")
-		(at 69.5 145.5)
+		(at 85.5625 142.5)
 		(descr "SOT, 3 Pin (JEDEC TO-236 Var AB https://www.jedec.org/document_search?search_api_views_fulltext=TO-236), generated with kicad-footprint-generator ipc_gullwing_generator.py")
 		(tags "SOT TO_SOT_SMD")
@@
 	(footprint "Resistor_SMD:R_1206_3216Metric"
 		(layer "F.Cu")
-		(at 137.4825 73.4)
+		(at 48.4625 140)
 		(descr "Resistor SMD 1206 (3216 Metric), square (rectangular) end terminal, IPC_7351 nominal, (Body size source: IPC-SM-782 page 72, https://www.pcb-3d.com/wordpress/wp-content/uploads/ipc-sm-782a_amendment_1_and_2.pdf), generated with kicad-footprint-generator")
 		(tags "resistor")

Commit message: making pcb
Parts:
- moved C5 138.9 mm to (69.0, 139.5)
- moved C6 138.6 mm to (69.0, 142.5)
- moved D5 136.1 mm to (54.6, 131.5)
- moved JP1 134.7 mm to (58.5, 145.3), turned to 90 degrees
- moved R8 132.7 mm to (73.5, 142.5)
- moved JP2 129.8 mm to (62.0, 145.3), turned to 90 degrees
- moved R3 129.7 mm to (53.9, 149.5), turned to 90 degrees
- moved R9 128.8 mm to (73.5, 139.5)
- moved R4 125.0 mm to (57.2, 149.5), turned to 90 degrees
- moved C11 123.0 mm to (47.3, 145.0)
- moved C4 122.8 mm to (50.8, 145.0)
- moved R5 120.4 mm to (60.5, 149.5), turned to 90 degrees
- moved C3 119.4 mm to (48.5, 127.5)
- moved C1 117.6 mm to (50.0, 123.5), turned to 90 degrees
- moved R6 115.7 mm to (63.8, 149.5), turned to 90 degrees
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Routing:
- net GND: track 0.00 -> 0.88 mm
- net Net-(Q1-B): track 0.00 -> 0.80 mm

Commit message: making pcb
Parts:
- removed D2, D3: LED, LED_SMD:LED_2010_5025Metric
- C3: footprint Capacitor_SMD:C_0805_2012Metric -> Capacitor_SMD:C_1206_3216Metric
- moved R4 111.1 mm to (154.0, 95.0), turned to 180 degrees
- moved C11 111.0 mm to (153.2, 112.0)
- moved SW3 109.7 mm to (153.5, 117.5)
- moved C4 109.5 mm to (151.7, 102.5)
- moved R3 104.4 mm to (150.0, 108.5)
- moved R6 104.1 mm to (154.0, 97.5), turned to 0 degrees
- moved JP1 103.6 mm to (150.0, 96.9), turned to -90 degrees
- moved R2 101.6 mm to (146.2, 90.5), turned to 180 degrees
- moved D5 100.1 mm to (144.5, 87.5), turned to 90 degrees
- moved C9 100.1 mm to (146.8, 87.5), turned to 90 degrees
- moved D4 99.8 mm to (138.6, 92.5), turned to 0 degrees
- moved C10 98.5 mm to (146.1, 92.5), turned to 180 degrees
- moved U4 98.0 mm to (152.5, 90.0)
- moved R12 96.8 mm to (133.5, 92.5), turned to 0 degrees
- moved C1 96.6 mm to (139.5, 87.2)
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Connections:
- R4 pad 2: Net-(D2-K) -> +3V3
- R5 pad 2: Net-(D3-K) -> +3V3
Routing:
- net GND: track 0.88 -> 268.0 mm, vias 0 -> 2
- net /EN: track 0.00 -> 106.8 mm, vias 0 -> 2
- net /IO9: track 0.00 -> 52.1 mm
- net +5V: track 0.00 -> 51.9 mm, vias 0 -> 2
- net /U0RXD: track 0.00 -> 46.9 mm
- net +3V3: track 0.00 -> 45.3 mm
- net /IO19: track 0.00 -> 36.7 mm
- net /IO18: track 0.00 -> 32.4 mm, vias 0 -> 1
- net /DTR: track 0.00 -> 30.9 mm, vias 0 -> 2
- net /U0TXD: track 0.00 -> 30.1 mm, vias 0 -> 2
- net /IO8: track 0.00 -> 26.8 mm
- net /IO7: track 0.00 -> 21.5 mm
- net /IO6: track 0.00 -> 20.1 mm
- net /IO4: track 0.00 -> 19.3 mm
- net /IO5: track 0.00 -> 19.2 mm
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
Commit message: updated design
Routing:
- net +3V3: track 45.3 -> 49.8 mm
- net GND: track 268.0 -> 270.3 mm, vias 2 -> 3
- net /EN: track 106.8 -> 106.7 mm, vias 2 -> 3
